Commit message: Update PID branch with current local workspace

File: install/w102_path_planning/share/w102_path_planning/urdf/w102_robot.urdf.xacro (robot description, xacro)
@@ -1,138 +1 @@
-<?xml version="1.0"?>
-<!--
-  W102 robot URDF for robot_state_publisher / RViz TF visualisation.
-  Matches the SDF model embedded in living_room.sdf.
-  Footprint: 27 in × 32 in  (0.686 m × 0.813 m)
-  Drive wheels: radius 0.10 m, separation 0.54 m
--->
-<robot name="w102" xmlns:xacro="http://www.ros.org/wiki/xacro">
-  <!-- ── Material colours ─────────────────────────────────────────────── -->
-  <material name="dark_grey"><color rgba="0.15 0.15 0.15 1"/></material>
-  <material name="orange">   <color rgba="1.0  0.5  0.0  1"/></material>
-  <material name="red">      <color rgba="0.8  0.2  0.0  1"/></material>
-  <material name="black">    <color rgba="0.1  0.1  0.1  1"/></material>
-  <!-- ── base_footprint (virtual ground link) ─────────────────────────── -->
-  <link name="base_footprint"/>
-  <joint name="base_footprint_joint" type="fixed">
-    <parent link="base_footprint"/>
-    <child  link="base_link"/>
-    <origin xyz="0 0 0.12" rpy="0 0 0"/>
-  </joint>
-  <!-- ── base_link ────────────────────────────────────────────────────── -->
-  <link name="base_link">
-    <visual>
-      <geometry><box size="0.686 0.813 0.20"/></geometry>
-      <material name="dark_grey"/>
-    </visual>
-    <collision>
-      <geometry><box size="0.686 0.813 0.20"/></geometry>
-    </collision>
-    <inertial>
-      <mass value="15.0"/>
-      <inertia ixx="0.35" ixy="0" ixz="0" iyy="0.50" iyz="0" izz="0.65"/>
-    </inertial>
-  </link>
-  <!-- Orange front bumper stripe -->
-  <link name="bumper_link">
-    <visual>
-      <geometry><box size="0.686 0.02 0.08"/></geometry>
-      <material name="orange"/>
-    </visual>
-  </link>
-  <joint name="bumper_joint" type="fixed">
-    <parent link="base_link"/>
-    <child  link="bumper_link"/>
-    <origin xyz="0 0.41 -0.05" rpy="0 0 0"/>
-  </joint>
-  <!-- Sensor tower (red cylinder on top) -->
-  <link name="sensor_tower">
-    <visual>
-      <geometry><cylinder radius="0.06" length="0.16"/></geometry>
-      <material name="red"/>
-    </visual>
-  </link>
-  <joint name="sensor_tower_joint" type="fixed">
-    <parent link="base_link"/>
-    <child  link="sensor_tower"/>
-    <origin xyz="0 0.1 0.18" rpy="0 0 0"/>
-  </joint>
-  <!-- ── Left drive wheel ─────────────────────────────────────────────── -->
-  <link name="left_wheel">
-    <visual>
-      <origin rpy="1.5708 0 0"/>
-      <geometry><cylinder radius="0.10" length="0.05"/></geometry>
-      <material name="black"/>
-    </visual>
-    <collision>
-      <origin rpy="1.5708 0 0"/>
-      <geometry><cylinder radius="0.10" length="0.05"/></geometry>
-    </collision>
-    <inertial>
-      <mass value="1.5"/>
-      <inertia ixx="0.0045" ixy="0" ixz="0" iyy="0.0045" iyz="0" izz="0.0075"/>
-    </inertial>
-  </link>
-  <joint name="left_wheel_joint" type="continuous">
-    <parent link="base_link"/>
-    <child  link="left_wheel"/>
-    <origin xyz="-0.27 0 -0.02" rpy="0 0 0"/>
-    <axis xyz="1 0 0"/>
-  </joint>
-  <!-- ── Right drive wheel ────────────────────────────────────────────── -->
-  <link name="right_wheel">
-    <visual>
-      <origin rpy="1.5708 0 0"/>
-      <geometry><cylinder radius="0.10" length="0.05"/></geometry>
-      <material name="black"/>
-    </visual>
-    <collision>
-      <origin rpy="1.5708 0 0"/>
-      <geometry><cylinder radius="0.10" length="0.05"/></geometry>
-    </collision>
-    <inertial>
-      <mass value="1.5"/>
-      <inertia ixx="0.0045" ixy="0" ixz="0" iyy="0.0045" iyz="0" izz="0.0075"/>
-    </inertial>
-  </link>
-  <joint name="right_wheel_joint" type="continuous">
-    <parent link="base_link"/>
-    <child  link="right_wheel"/>
-    <origin xyz="0.27 0 -0.02" rpy="0 0 0"/>
-    <axis xyz="1 0 0"/>
-  </joint>
-  <!-- ── Front caster ──────────────────────────────────────────────────── -->
-  <link name="caster_wheel">
-    <visual>
-      <geometry><sphere radius="0.05"/></geometry>
-      <material name="dark_grey"/>
-    </visual>
-    <collision>
-      <geometry><sphere radius="0.05"/></geometry>
-    </collision>
-    <inertial>
-      <mass value="0.3"/>
-      <inertia ixx="0.0003" ixy="0" ixz="0" iyy="0.0003" iyz="0" izz="0.0003"/>
-    </inertial>
-  </link>
-  <joint name="caster_joint" type="fixed">
-    <parent link="base_link"/>
-    <child  link="caster_wheel"/>
-    <origin xyz="0 0.36 -0.07" rpy="0 0 0"/>
-  </joint>
-  <!-- ── Rear caster ───────────────────────────────────────────────────── -->
-  <link name="caster_rear">
-    <visual>
-      <geometry><sphere radius="0.05"/></geometry>
-      <material name="dark_grey"/>
-    </visual>
-    <inertial>
-      <mass value="0.3"/>
-      <inertia ixx="0.0003" ixy="0" ixz="0" iyy="0.0003" iyz="0" izz="0.0003"/>
-    </inertial>
-  </link>
-  <joint name="caster_rear_joint" type="fixed">
-    <parent link="base_link"/>
-    <child  link="caster_rear"/>
-    <origin xyz="0 -0.36 -0.07" rpy="0 0 0"/>
-  </joint>
-</robot>
+/home/myy/CTI_One_interview/build/w102_path_planning/urdf/w102_robot.urdf.xacro
