Commit message: Fix Gazebo robot pose mismatch with ROS odometry and RViz

File: src/w102_path_planning/urdf/w102_robot.urdf.xacro (robot description, xacro)
@@ -12,12 +12,5 @@
   <material name="red">      <color rgba="0.8  0.2  0.0  1"/></material>
   <material name="black">    <color rgba="0.1  0.1  0.1  1"/></material>
-  <!-- ── base_footprint (virtual ground link) ─────────────────────────── -->
-  <link name="base_footprint"/>
-  <joint name="base_footprint_joint" type="fixed">
-    <parent link="base_footprint"/>
-    <child  link="base_link"/>
-    <origin xyz="0 0 0.12" rpy="0 0 0"/>
-  </joint>
-  <!-- ── base_link ────────────────────────────────────────────────────── -->
+  <!-- ── base_link (root link — OdometryPublisher in SDF provides odom→base_link) ── -->
   <link name="base_link">
     <visual>

Commit message: Fix TF conflict: DiffDrive child_frame_id base_link->base_footprint, restore URDF base_footprint

File: src/w102_path_planning/urdf/w102_robot.urdf.xacro (robot description, xacro)
@@ -12,5 +12,12 @@
   <material name="red">      <color rgba="0.8  0.2  0.0  1"/></material>
   <material name="black">    <color rgba="0.1  0.1  0.1  1"/></material>
-  <!-- ── base_link (root link — OdometryPublisher in SDF provides odom→base_link) ── -->
+  <!-- ── base_footprint (virtual ground link; DiffDrive publishes odom→base_footprint) ── -->
+  <link name="base_footprint"/>
+  <joint name="base_footprint_joint" type="fixed">
+    <parent link="base_footprint"/>
+    <child  link="base_link"/>
+    <origin xyz="0 0 0.12" rpy="0 0 0"/>
+  </joint>
+  <!-- ── base_link ────────────────────────────────────────────────────── -->
   <link name="base_link">
     <visual>

Commit message: Fix orientation mismatch: forward=+X (axis Y wheels), spawn yaw=0, visual markers aligned

File: src/w102_path_planning/urdf/w102_robot.urdf.xacro (robot description, xacro)
@@ -22,9 +22,9 @@
   <link name="base_link">
     <visual>
-      <geometry><box size="0.686 0.813 0.20"/></geometry>
+      <geometry><box size="0.813 0.686 0.20"/></geometry>
       <material name="dark_grey"/>
     </visual>
     <collision>
-      <geometry><box size="0.686 0.813 0.20"/></geometry>
+      <geometry><box size="0.813 0.686 0.20"/></geometry>
     </collision>
     <inertial>
@@ -36,5 +36,5 @@
   <link name="bumper_link">
     <visual>
-      <geometry><box size="0.686 0.02 0.08"/></geometry>
+      <geometry><box size="0.02 0.686 0.08"/></geometry>
       <material name="orange"/>
     </visual>
@@ -43,5 +43,5 @@
     <parent link="base_link"/>
     <child  link="bumper_link"/>
-    <origin xyz="0 0.41 -0.05" rpy="0 0 0"/>
+    <origin xyz="0.41 0 -0.05" rpy="0 0 0"/>
   </joint>
   <!-- Sensor tower (red cylinder on top) -->
@@ -55,5 +55,5 @@
     <parent link="base_link"/>
     <child  link="sensor_tower"/>
-    <origin xyz="0 0.1 0.18" rpy="0 0 0"/>
+    <origin xyz="0.1 0 0.18" rpy="0 0 0"/>
   </joint>
   <!-- ── Left drive wheel ─────────────────────────────────────────────── -->
@@ -76,6 +76,6 @@
     <parent link="base_link"/>
     <child  link="left_wheel"/>
-    <origin xyz="-0.27 0 -0.02" rpy="0 0 0"/>
-    <axis xyz="1 0 0"/>
+    <origin xyz="0 0.27 -0.02" rpy="0 0 0"/>
+    <axis xyz="0 1 0"/>
   </joint>
   <!-- ── Right drive wheel ────────────────────────────────────────────── -->
@@ -98,6 +98,6 @@
     <parent link="base_link"/>
     <child  link="right_wheel"/>
-    <origin xyz="0.27 0 -0.02" rpy="0 0 0"/>
-    <axis xyz="1 0 0"/>
+    <origin xyz="0 -0.27 -0.02" rpy="0 0 0"/>
+    <axis xyz="0 1 0"/>
   </joint>
   <!-- ── Front caster ──────────────────────────────────────────────────── -->
@@ -118,5 +118,5 @@
     <parent link="base_link"/>
     <child  link="caster_wheel"/>
-    <origin xyz="0 0.36 -0.07" rpy="0 0 0"/>
+    <origin xyz="0.36 0 -0.07" rpy="0 0 0"/>
   </joint>
   <!-- ── Rear caster ───────────────────────────────────────────────────── -->
@@ -134,5 +134,5 @@
     <parent link="base_link"/>
     <child  link="caster_rear"/>
-    <origin xyz="0 -0.36 -0.07" rpy="0 0 0"/>
+    <origin xyz="-0.36 0 -0.07" rpy="0 0 0"/>
   </joint>
 </robot>

Commit message: Revert drivetrain geometry to working convention (axis X, spawn yaw=pi/2)

File: src/w102_path_planning/urdf/w102_robot.urdf.xacro (robot description, xacro)
@@ -22,9 +22,9 @@
   <link name="base_link">
     <visual>
-      <geometry><box size="0.813 0.686 0.20"/></geometry>
+      <geometry><box size="0.686 0.813 0.20"/></geometry>
       <material name="dark_grey"/>
     </visual>
     <collision>
-      <geometry><box size="0.813 0.686 0.20"/></geometry>
+      <geometry><box size="0.686 0.813 0.20"/></geometry>
     </collision>
     <inertial>
@@ -36,5 +36,5 @@
   <link name="bumper_link">
     <visual>
-      <geometry><box size="0.02 0.686 0.08"/></geometry>
+      <geometry><box size="0.686 0.02 0.08"/></geometry>
       <material name="orange"/>
     </visual>
@@ -43,5 +43,5 @@
     <parent link="base_link"/>
     <child  link="bumper_link"/>
-    <origin xyz="0.41 0 -0.05" rpy="0 0 0"/>
+    <origin xyz="0 0.41 -0.05" rpy="0 0 0"/>
   </joint>
   <!-- Sensor tower (red cylinder on top) -->
@@ -55,5 +55,5 @@
     <parent link="base_link"/>
     <child  link="sensor_tower"/>
-    <origin xyz="0.1 0 0.18" rpy="0 0 0"/>
+    <origin xyz="0 0.1 0.18" rpy="0 0 0"/>
   </joint>
   <!-- ── Left drive wheel ─────────────────────────────────────────────── -->
@@ -76,6 +76,6 @@
     <parent link="base_link"/>
     <child  link="left_wheel"/>
-    <origin xyz="0 0.27 -0.02" rpy="0 0 0"/>
-    <axis xyz="0 1 0"/>
+    <origin xyz="-0.27 0 -0.02" rpy="0 0 0"/>
+    <axis xyz="1 0 0"/>
   </joint>
   <!-- ── Right drive wheel ────────────────────────────────────────────── -->
@@ -98,6 +98,6 @@
     <parent link="base_link"/>
     <child  link="right_wheel"/>
-    <origin xyz="0 -0.27 -0.02" rpy="0 0 0"/>
-    <axis xyz="0 1 0"/>
+    <origin xyz="0.27 0 -0.02" rpy="0 0 0"/>
+    <axis xyz="1 0 0"/>
   </joint>
   <!-- ── Front caster ──────────────────────────────────────────────────── -->
@@ -118,5 +118,5 @@
     <parent link="base_link"/>
     <child  link="caster_wheel"/>
-    <origin xyz="0.36 0 -0.07" rpy="0 0 0"/>
+    <origin xyz="0 0.36 -0.07" rpy="0 0 0"/>
   </joint>
   <!-- ── Rear caster ───────────────────────────────────────────────────── -->
@@ -134,5 +134,5 @@
     <parent link="base_link"/>
     <child  link="caster_rear"/>
-    <origin xyz="-0.36 0 -0.07" rpy="0 0 0"/>
+    <origin xyz="0 -0.36 -0.07" rpy="0 0 0"/>
   </joint>
 </robot>

Commit message: Visual-only fix: spawn yaw=0, bumper/tower face +X, drivetrain physics unchanged

File: src/w102_path_planning/urdf/w102_robot.urdf.xacro (robot description, xacro)
@@ -36,5 +36,5 @@
   <link name="bumper_link">
     <visual>
-      <geometry><box size="0.686 0.02 0.08"/></geometry>
+      <geometry><box size="0.02 0.686 0.08"/></geometry>
       <material name="orange"/>
     </visual>
@@ -43,5 +43,5 @@
     <parent link="base_link"/>
     <child  link="bumper_link"/>
-    <origin xyz="0 0.41 -0.05" rpy="0 0 0"/>
+    <origin xyz="0.41 0 -0.05" rpy="0 0 0"/>
   </joint>
   <!-- Sensor tower (red cylinder on top) -->
@@ -55,5 +55,5 @@
     <parent link="base_link"/>
     <child  link="sensor_tower"/>
-    <origin xyz="0 0.1 0.18" rpy="0 0 0"/>
+    <origin xyz="0.1 0 0.18" rpy="0 0 0"/>
   </joint>
   <!-- ── Left drive wheel ─────────────────────────────────────────────── -->

Commit message: fix: correct wheel positions, joint axes, and caster placement for diff-drive
Drive wheels moved from x=±0.27 to y=±0.27 so they sit on the left/right
sides of the +X-facing robot. Joint revolute axes changed from X to Y so
the DiffDrive plugin rolls the wheels forward. Casters moved from y=±0.36
to x=±0.36 (front/rear). Matching changes in URDF xacro for TF consistency.
Fixed misleading launch file comment about paused start.

File: src/w102_path_planning/urdf/w102_robot.urdf.xacro (robot description, xacro)
@@ -76,6 +76,6 @@
     <parent link="base_link"/>
     <child  link="left_wheel"/>
-    <origin xyz="-0.27 0 -0.02" rpy="0 0 0"/>
-    <axis xyz="1 0 0"/>
+    <origin xyz="0 0.27 -0.02" rpy="0 0 0"/>
+    <axis xyz="0 1 0"/>
   </joint>
   <!-- ── Right drive wheel ────────────────────────────────────────────── -->
@@ -98,6 +98,6 @@
     <parent link="base_link"/>
     <child  link="right_wheel"/>
-    <origin xyz="0.27 0 -0.02" rpy="0 0 0"/>
-    <axis xyz="1 0 0"/>
+    <origin xyz="0 -0.27 -0.02" rpy="0 0 0"/>
+    <axis xyz="0 1 0"/>
   </joint>
   <!-- ── Front caster ──────────────────────────────────────────────────── -->
@@ -118,5 +118,5 @@
     <parent link="base_link"/>
     <child  link="caster_wheel"/>
-    <origin xyz="0 0.36 -0.07" rpy="0 0 0"/>
+    <origin xyz="0.36 0 -0.07" rpy="0 0 0"/>
   </joint>
   <!-- ── Rear caster ───────────────────────────────────────────────────── -->
@@ -134,5 +134,5 @@
     <parent link="base_link"/>
     <child  link="caster_rear"/>
-    <origin xyz="0 -0.36 -0.07" rpy="0 0 0"/>
+    <origin xyz="-0.36 0 -0.07" rpy="0 0 0"/>
   </joint>
 </robot>
