Commit message: Fix robot forward direction: wheels on Y-axis so yaw=0 faces +X, matching nav atan2 convention
Drive wheels moved from X=±0.27 (axis X) to Y=±0.27 (axis Y) in both
living_room.sdf and w102_robot.urdf.xacro. Casters moved from Y=±0.36
to X=±0.36. Base box X/Y swapped (0.813×0.686). This makes the robot
physically face and move in +X at yaw=0, aligning Gazebo motion with the
2D path-sim trajectory (S→R1 east, R1→R2 north, R2→G northwest).

Co-Authored-By: Claude Sonnet 4.6 <noreply@anthropic.com>

File: src/w102_path_planning/urdf/w102_robot.urdf.xacro (robot description, xacro)
@@ -22,13 +22,13 @@
   <link name="base_link">
     <visual>
-      <geometry><box size="0.686 0.813 0.20"/></geometry>
+      <geometry><box size="0.813 0.686 0.20"/></geometry>
       <material name="dark_grey"/>
     </visual>
     <collision>
-      <geometry><box size="0.686 0.813 0.20"/></geometry>
+      <geometry><box size="0.813 0.686 0.20"/></geometry>
     </collision>
     <inertial>
       <mass value="15.0"/>
-      <inertia ixx="0.35" ixy="0" ixz="0" iyy="0.50" iyz="0" izz="0.65"/>
+      <inertia ixx="0.50" ixy="0" ixz="0" iyy="0.35" iyz="0" izz="0.65"/>
     </inertial>
   </link>
@@ -76,6 +76,6 @@
     <parent link="base_link"/>
     <child  link="left_wheel"/>
-    <origin xyz="-0.27 0 -0.02" rpy="0 0 0"/>
-    <axis xyz="1 0 0"/>
+    <origin xyz="0 0.27 -0.02" rpy="0 0 0"/>
+    <axis xyz="0 1 0"/>
   </joint>
   <!-- ── Right drive wheel ────────────────────────────────────────────── -->
@@ -98,6 +98,6 @@
     <parent link="base_link"/>
     <child  link="right_wheel"/>
-    <origin xyz="0.27 0 -0.02" rpy="0 0 0"/>
-    <axis xyz="1 0 0"/>
+    <origin xyz="0 -0.27 -0.02" rpy="0 0 0"/>
+    <axis xyz="0 1 0"/>
   </joint>
   <!-- ── Front caster ──────────────────────────────────────────────────── -->
@@ -118,5 +118,5 @@
     <parent link="base_link"/>
     <child  link="caster_wheel"/>
-    <origin xyz="0 0.36 -0.07" rpy="0 0 0"/>
+    <origin xyz="0.36 0 -0.07" rpy="0 0 0"/>
   </joint>
   <!-- ── Rear caster ───────────────────────────────────────────────────── -->
@@ -134,5 +134,5 @@
     <parent link="base_link"/>
     <child  link="caster_rear"/>
-    <origin xyz="0 -0.36 -0.07" rpy="0 0 0"/>
+    <origin xyz="-0.36 0 -0.07" rpy="0 0 0"/>
   </joint>
 </robot>

Commit message: Fix ros_gz_bridge: use positional arguments instead of config_file parameter
ros_gz_bridge 2.1.15 (Kilted) does not resolve 'config_file' as a file
path when passed as a ROS parameter — it attempts to parse the path string
as inline YAML, producing "top level must be a YAML sequence" errors and
leaving /odom unbridged so the nav node never receives odometry.

Switch to positional CLI arguments which are supported in all versions.

Co-Authored-By: Claude Sonnet 4.6 <noreply@anthropic.com>

File: src/w102_path_planning/urdf/w102_robot.urdf.xacro (robot description, xacro)
@@ -12,5 +12,5 @@
   <material name="red">      <color rgba="0.8  0.2  0.0  1"/></material>
   <material name="black">    <color rgba="0.1  0.1  0.1  1"/></material>
-  <!-- ── base_footprint (virtual ground link) ─────────────────────────── -->
+  <!-- ── base_footprint (virtual ground link; DiffDrive publishes odom→base_footprint) ── -->
   <link name="base_footprint"/>
   <joint name="base_footprint_joint" type="fixed">
@@ -36,5 +36,5 @@
   <link name="bumper_link">
     <visual>
-      <geometry><box size="0.686 0.02 0.08"/></geometry>
+      <geometry><box size="0.02 0.686 0.08"/></geometry>
       <material name="orange"/>
     </visual>
@@ -43,5 +43,5 @@
     <parent link="base_link"/>
     <child  link="bumper_link"/>
-    <origin xyz="0 0.41 -0.05" rpy="0 0 0"/>
+    <origin xyz="0.41 0 -0.05" rpy="0 0 0"/>
   </joint>
   <!-- Sensor tower (red cylinder on top) -->
@@ -55,5 +55,5 @@
     <parent link="base_link"/>
     <child  link="sensor_tower"/>
-    <origin xyz="0 0.1 0.18" rpy="0 0 0"/>
+    <origin xyz="0.1 0 0.18" rpy="0 0 0"/>
   </joint>
   <!-- ── Left drive wheel ─────────────────────────────────────────────── -->
@@ -76,6 +76,6 @@
     <parent link="base_link"/>
     <child  link="left_wheel"/>
-    <origin xyz="-0.27 0 -0.02" rpy="0 0 0"/>
-    <axis xyz="1 0 0"/>
+    <origin xyz="0 0.27 -0.02" rpy="0 0 0"/>
+    <axis xyz="0 1 0"/>
   </joint>
   <!-- ── Right drive wheel ────────────────────────────────────────────── -->
@@ -98,6 +98,6 @@
     <parent link="base_link"/>
     <child  link="right_wheel"/>
-    <origin xyz="0.27 0 -0.02" rpy="0 0 0"/>
-    <axis xyz="1 0 0"/>
+    <origin xyz="0 -0.27 -0.02" rpy="0 0 0"/>
+    <axis xyz="0 1 0"/>
   </joint>
   <!-- ── Front caster ──────────────────────────────────────────────────── -->
@@ -118,5 +118,5 @@
     <parent link="base_link"/>
     <child  link="caster_wheel"/>
-    <origin xyz="0 0.36 -0.07" rpy="0 0 0"/>
+    <origin xyz="0.36 0 -0.07" rpy="0 0 0"/>
   </joint>
   <!-- ── Rear caster ───────────────────────────────────────────────────── -->
@@ -134,5 +134,5 @@
     <parent link="base_link"/>
     <child  link="caster_rear"/>
-    <origin xyz="0 -0.36 -0.07" rpy="0 0 0"/>
+    <origin xyz="-0.36 0 -0.07" rpy="0 0 0"/>
   </joint>
 </robot>
